File: eagle/sonnette/test.sch (EAGLE design)
At the start: 14 parts, among them IC1 7805TV, IC2 4066N, Q1 60V/32A/35mΩ

Commit message: update schema for receiver
Parts:
- added C3: 33uF, SparkFun-Capacitors:0.1UF-KIT-EZ-50V-20%
- added C4: 0.47uF, SparkFun-Capacitors:0.1UF-KIT-EZ-50V-20%
- added C5, C6, C7: 10uF, SparkFun-Capacitors:10UF-POLAR-RADIAL-2.5MM-25V-20%
- added FM_TX, JP7: (no value), pinhead:PINHD-1X4
- added IC3: LM3840, linear:7805TV
- added J1: POWER_JACK, SparkFun-Connectors:POWER_JACK
- added JP3, JP4: (no value), pinhead:PINHD-1X5
- added JP5, JP6: (no value), pinhead:PINHD-1X6
- added JP8: (no value), pinhead:PINHD-1X2
- added LCD1: LCD-16X2SILK, SparkFun-Displays:LCD-16X2SILK
- added LS1: SPEAKER, SparkFun-Electromechanical:SPEAKER
- added Q2: IRFZ44N, SparkFun-DiscreteSemi:MOSFET-NCH-FQP30N06L
- added R10, R12, R13, R5: 4.7k, SparkFun-Resistors:1KOHM-HORIZ-1/4W-1%
- added R11, R14, R6, R9: 1k, SparkFun-Resistors:1KOHM-HORIZ-1/4W-1%
- added R15: (no value), rcl:POTENTIOMETER_PT-10
- added R3, R4, R7, R8: 10k, SparkFun-Resistors:1KOHM-HORIZ-1/4W-1%
- added S1: MOMENTARY-SWITCH-SPST-PTH-6.0MM, SparkFun-Switches:MOMENTARY-SWITCH-SPST-PTH-6.0MM
- added T1: 2N2222, adafruit:2N2222
- Q1: value 60V/32A/35mΩ -> IRFZ44N
Connections:
- new net 3V3_REGU: C3.1, IC3.VO, JP3.1, JP6.4
- new net 5V_ON: Q2.G, R6.2
- new net 5V_REGU: C4.1, FM_TX.2, IC3.VI, JP5.4, Q2.S, R8.1
- new net AUDIO_OUT1: JP4.2, JP4.3
- new net AUDIO_OUT2: C5.-, C7.-, U$1.D12
- new net AUDIO_SELECT: IC2C.C, R7.2, U$1.D13
- new net E: LCD1.E, U$1.D9
- new net N$10: R5.1, U$2.ANT, U$2.DATA
- new net N$11: JP3.5, JP6.6
- new net N$12: JP3.4, JP6.5
- new net N$13: R7.1, T1.B
- new net N$14: IC2C.A, R10.2
- new net N$15: C5.+, R10.1, R9.1
- new net N$16: IC2B.C, R8.2, T1.C
- new net N$17: IC2B.A, R12.2
- new net N$18: C7.+, R11.1, R12.1
- new net N$19: JP8.1, LS1.+
- new net N$20: JP7.3, JP7.4
- new net N$21: C6.-, IC2B.B, IC2C.B, R13.2
- new net N$22: C6.+, JP7.2
- new net N$23: R13.1
- new net N$24: JP8.2, LS1.-
- new net N$25: J1.GND, J1.GNDBREAK
- new net N$26: S1.2, U$1.D5
- new net N$27: LCD1.DB7, U$1.A0
- new net N$28: LCD1.DB6, U$1.A1
- new net N$29: LCD1.DB5, U$1.A2
- new net N$30: LCD1.DB4, U$1.A3
- new net N$31: LCD1.VDD
- new net N$32: LCD1.VSS, R15.2
- new net N$34: LCD1.A, R14.2
- new net N$36: LCD1.VO, R15.3
- new net N$8: IC2A.C, R4.1
- new net N$9: IC2A.B, R5.2
- new net RS: LCD1.RS, U$1.D8
- new net SCL: FM_TX.4, JP5.5, U$1.A5
- new net SDA: FM_TX.3, JP5.6, U$1.A4
- net 12V: now also IC2P.VDD, JP7.1, R3.2; no longer IC2A.A
- net GND: now also C3.2, C4.2, DC1.-VIN1, DC1.-VOUT1, FM_TX.1, IC2P.VSS, IC3.GND, JP4.1, JP5.3, JP6.3, LCD1.K, R11.2, T1.E
- net N$6: now also J1.PWR
- net N$7: now also DC1.+VIN1, Q1.S; no longer DC1.-VIN1, Q1.D
- net RF_TX: now also R4.2, U$1.D7; no longer IC2A.B, IC2A.C, U$1.D8, U$2.ANT, U$2.DATA
- net VCC: now also Q1.D, Q2.D, R14.1, R15.1; no longer DC1.+VIN1
Other:
- moved on the sheet: C1, C2, DC1, IC1, IC2A, IC2B, IC2C, IC2D, Q1, R2

Commit message: update
Connections:
- removed net N$13: R7.1, T1.B
- net AUDIO_SELECT: now also R7.1, T1.B
Changed lines of the file:
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@@
 <layer number="91" name="Nets" color="2" fill="1" visible="yes" active="yes"/>
 <layer number="92" name="Busses" color="1" fill="1" visible="yes" active="yes"/>
-<layer number="93" name="Pins" color="2" fill="1" visible="no" active="yes"/>
+<layer number="93" name="Pins" color="2" fill="1" visible="yes" active="yes"/>
 <layer number="94" name="Symbols" color="4" fill="1" visible="yes" active="yes"/>
 <layer number="95" name="Names" color="7" fill="1" visible="yes" active="yes"/>
@@
 <instance part="SUPPLY4" gate="G$1" x="-1447.8" y="579.12"/>
 <instance part="GND20" gate="1" x="-1440.18" y="579.12" rot="R270"/>
-<instance part="GND21" gate="1" x="-1437.64" y="568.96" rot="R270"/>
+<instance part="GND21" gate="1" x="-1440.18" y="568.96" rot="R270"/>
 <instance part="GND22" gate="1" x="-1430.02" y="535.94"/>
 <instance part="R14" gate="G$1" x="-1440.18" y="541.02"/>
@@
 <wire x1="-1539.24" y1="528.32" x2="-1539.24" y2="525.78" width="0.1524" layer="91"/>
 </segment>
+<segment>
+<pinref part="GND21" gate="1" pin="GND"/>
+<wire x1="-1430.02" y1="568.96" x2="-1437.64" y2="568.96" width="0.1524" layer="91"/>
+</segment>
 </net>
 <net name="N$2" class="0">
@@
 </segment>
 </net>
-<net name="N$13" class="0">
-<segment>
-<pinref part="R7" gate="G$1" pin="1"/>
-<pinref part="T1" gate="G$1" pin="B"/>
-<wire x1="-1866.9" y1="579.12" x2="-1859.28" y2="579.12" width="0.1524" layer="91"/>
-</segment>
-</net>
 <net name="AUDIO_SELECT" class="0">
 <segment>
@@
 </segment>
 <segment>
+<pinref part="IC2" gate="C" pin="C"/>
+<wire x1="-1765.3" y1="558.8" x2="-1864.36" y2="558.8" width="0.1524" layer="91"/>
+<pinref part="R7" gate="G$1" pin="1"/>
+<pinref part="T1" gate="G$1" pin="B"/>
+<wire x1="-1866.9" y1="579.12" x2="-1864.36" y2="579.12" width="0.1524" layer="91"/>
+<wire x1="-1864.36" y1="579.12" x2="-1859.28" y2="579.12" width="0.1524" layer="91"/>
+<wire x1="-1864.36" y1="558.8" x2="-1864.36" y2="579.12" width="0.1524" layer="91"/>
+<junction x="-1864.36" y="579.12"/>
+</segment>
+<segment>
 <pinref part="R7" gate="G$1" pin="2"/>
-<wire x1="-1877.06" y1="579.12" x2="-1884.68" y2="579.12" width="0.1524" layer="91"/>
+<wire x1="-1877.06" y1="579.12" x2="-1894.84" y2="579.12" width="0.1524" layer="91"/>
 <label x="-1899.92" y="579.12" size="1.778" layer="95"/>
-<wire x1="-1884.68" y1="579.12" x2="-1894.84" y2="579.12" width="0.1524" layer="91"/>
-<wire x1="-1884.68" y1="558.8" x2="-1884.68" y2="579.12" width="0.1524" layer="91"/>
-<junction x="-1884.68" y="579.12"/>
-<pinref part="IC2" gate="C" pin="C"/>
-<wire x1="-1765.3" y1="558.8" x2="-1884.68" y2="558.8" width="0.1524" layer="91"/>
 </segment>
 </net>
@@
 </segment>
 </net>
-<net name="N$33" class="0">
-<segment>
-<wire x1="-1427.48" y1="568.96" x2="-1435.1" y2="568.96" width="0.1524" layer="91"/>
-</segment>
-</net>
 <net name="RS" class="0">
 <segment>
@@
 </sheet>
 </sheets>
+<errors>
+</errors>
 </schematic>
 </drawing>

Commit message: updated eagle schema
Parts:
- added C10, C11, C12, C13, C8, C9: 0.1uF, SparkFun-Capacitors:0.1UF-KIT-EZ-50V-20%
Connections:
- new net N$13: R6.1, U$1.D11
- net 12V: now also C13.1, C8.1
- net 3V3_REGU: now also C10.2
- net 5V_REGU: now also C11.2
- net AUDIO_OUT1: now also C7.-
- net AUDIO_OUT2: no longer C7.-
- net GND: now also C10.1, C11.1, C12.2, C13.2, C8.2, J1.GND, J1.GNDBREAK, LCD1.R/W, R9.2, S1.1
- net N$25: now also IC2A.A, R3.1; no longer J1.GND, J1.GNDBREAK
- net VCC: now also C12.1
Other:
- note added: "433MHz RX"
- note added: "433MHz TX"
- note added: "ARDUINO + LCD"
- note added: "AUDIO_MIX"
- note added: "FM RX"
- note added: "FM TX"
- note added: "Level shifter"
- note added: "POWER SUPPLY"
- moved on the sheet: C1, C2, C3, C4, C5, C6, C7, DC1, FM_TX, IC1, IC2A, IC2B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
